File: pcb/CoCoFlash_v1.04c.sch (EAGLE design)
At the start: 92 parts, among them IC1 ST95P08M, IC3 XC95144XLTQG100, IC4 '574, IC5 '574, IC6 LM4558D, IC8 AZ1117CH-3.3, Q1 2n7002, X1 EXPANSION_PORT_COCO, X2 SJ1-3525N

Commit message: Small PCB cleanup
Parts:
- added PAK: PROGRAM_PAK, coco:PROGRAM_PAK
Changed lines of the file:
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@@
 <?xml version="1.0" encoding="utf-8"?>
 <!DOCTYPE eagle SYSTEM "eagle.dtd">
-<eagle version="7.6.0">
+<eagle version="7.7.0">
 <drawing>
 <settings>
@@
 <layer number="106" name="BGA-Top" color="4" fill="1" visible="yes" active="yes"/>
 <layer number="107" name="BD-Top" color="5" fill="1" visible="yes" active="yes"/>
+<layer number="110" name="OldCocoCase" color="7" fill="1" visible="yes" active="yes"/>
+<layer number="111" name="NewCocoCase" color="7" fill="1" visible="yes" active="yes"/>
 <layer number="116" name="Patch_BOT" color="9" fill="4" visible="yes" active="yes"/>
 <layer number="121" name="_tsilk" color="7" fill="1" visible="yes" active="yes"/>
@@
 <part name="SUPPLY3" library="supply2" deviceset="GND" device=""/>
 <part name="SUPPLY4" library="supply2" deviceset="GND" device=""/>
+<part name="PAK" library="coco" deviceset="PROGRAM_PAK" device=""/>
 </parts>
 <sheets>
@@
 <attribute name="VALUE" x="244.602" y="13.97" size="1.778" layer="96" rot="R90"/>
 </instance>
+<instance part="PAK" gate="A" x="-81.28" y="-172.72"/>
 </instances>
 <busses>
